File: AI Camera/board/board.brd (EAGLE design)
At the start: 46 x 47 mm, 23 parts

Commit message: More woek on the AI Camera PCB
Parts:
- moved ETH_+12V(2) 5.08 mm to (48.9, 11.4)
- moved ETH_GND(1) 5.08 mm to (46.4, 11.4)
- moved ETH_GND(3) 5.08 mm to (43.8, 11.4)
- moved ETH_SDA 5.08 mm to (41.3, 11.4)
- moved ETH_+12V(1) 5.08 mm to (50.2, 14.0)
- moved ETH_+12V(3) 5.08 mm to (47.6, 14.0)
- moved ETH_GND(2) 5.08 mm to (45.1, 14.0)
- moved ETH_SCL 5.08 mm to (42.5, 14.0)
Connections:
- removed net N$8: B1.1, ETH_SDA.1
- new net N$1: B1.5, ETH_SDA.1
- net N$3: now also B1.1, HSK_TX.1; no longer B1.13, HSK_RX.1
- net N$4: now also B1.2, HSK_RX.1; no longer B1.12, HSK_TX.1
- net N$5: now also B1.7; no longer B1.6
- net N$9: now also B1.6; no longer B1.2
Routing:
- net N$8: track 53.5 -> 0.00 mm
- net N$1: track 0.00 -> 41.2 mm
- net N$3: track 21.9 -> 57.1 mm
- net N$6: track 112.2 -> 122.4 mm
- net N$9: track 44.1 -> 34.2 mm
- net N$2: track 18.8 -> 20.9 mm
- net N$4: track 75.8 -> 77.5 mm
Other:
- board size 46 x 47 mm -> 45.4 x 77.5 mm
