File: Switch Board/board/board.brd (EAGLE design)
At the start: 100 x 80 mm, 17 parts

Commit message: Updated cart checklist and created printable copy of the board
Other:
- board size 100 x 80 mm -> 37.8 x 49.5 mm
Changed lines of the file:
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@@
 <board>
 <plain>
-<wire x1="0" y1="0" x2="100" y2="0" width="0" layer="20"/>
-<wire x1="100" y1="0" x2="100" y2="80" width="0" layer="20"/>
-<wire x1="100" y1="80" x2="0" y2="80" width="0" layer="20"/>
-<wire x1="0" y1="80" x2="0" y2="0" width="0" layer="20"/>
+<wire x1="15.24" y1="17.78" x2="53.01" y2="17.78" width="0" layer="20"/>
+<wire x1="53.01" y1="17.78" x2="53.01" y2="67.3" width="0" layer="20"/>
+<wire x1="53.01" y1="67.3" x2="15.24" y2="67.3" width="0" layer="20"/>
+<wire x1="15.24" y1="67.3" x2="15.24" y2="17.78" width="0" layer="20"/>
 </plain>
 <attributes>
