File: Auxiliary Sensors/board/board.sch (EAGLE design)
At the start: 61 parts

Commit message: Adding the thing to measure voltages
Parts:
- added VCC_MESURE: (no value), wirepad:2,15/1,0
Connections:
- new net N$12: VCC_MESURE.P
- new net N$4: B1.A0
Changed lines of the file:
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@@
 <?xml version="1.0" encoding="utf-8"?>
 <!DOCTYPE eagle SYSTEM "eagle.dtd">
-<eagle version="9.2.2">
+<eagle version="9.6.2">
 <drawing>
 <settings>
@@
 <part name="GF_AD0" library="wirepad" library_urn="urn:adsk.eagle:library:412" deviceset="2,15/1,0" device="" package3d_urn="urn:adsk.eagle:package:30831/1"/>
 <part name="GF_INT" library="wirepad" library_urn="urn:adsk.eagle:library:412" deviceset="2,15/1,0" device="" package3d_urn="urn:adsk.eagle:package:30831/1"/>
+<part name="R1" library="docu-dummy" library_urn="urn:adsk.eagle:library:215" deviceset="R" device="" value="BIG"/>
+<part name="VCC_MESURE" library="wirepad" library_urn="urn:adsk.eagle:library:412" deviceset="2,15/1,0" device="" package3d_urn="urn:adsk.eagle:package:30831/1"/>
 </parts>
 <sheets>
@@
 <attribute name="NAME" x="67.8942" y="64.643" size="1.778" layer="95" rot="R270"/>
 <attribute name="VALUE" x="62.738" y="64.643" size="1.778" layer="96" rot="R270"/>
+</instance>
+<instance part="R1" gate="G$1" x="50.8" y="25.4" smashed="yes"/>
+<instance part="VCC_MESURE" gate="1" x="0" y="12.7" smashed="yes">
+<attribute name="NAME" x="-1.143" y="14.5542" size="1.778" layer="95"/>
+<attribute name="VALUE" x="-1.143" y="9.398" size="1.778" layer="96"/>
 </instance>
 </instances>
@@
 </segment>
 </net>
+<net name="N$4" class="0">
+<segment>
+<pinref part="B1" gate="G$1" pin="A0"/>
+<wire x1="45.72" y1="25.4" x2="43.18" y2="25.4" width="0.1524" layer="91"/>
+</segment>
+</net>
+<net name="N$12" class="0">
+<segment>
+<wire x1="55.88" y1="25.4" x2="55.88" y2="2.54" width="0.1524" layer="91"/>
+<pinref part="VCC_MESURE" gate="1" pin="P"/>
+<wire x1="55.88" y1="2.54" x2="2.54" y2="2.54" width="0.1524" layer="91"/>
+<wire x1="2.54" y1="2.54" x2="2.54" y2="12.7" width="0.1524" layer="91"/>
+</segment>
+</net>
